File: Design/pcb/buck_bidireccional/buck_bidireccional.kicad_pcb (KiCad board)
At the start: 2 copper layers, 85 x 60 mm, 25 parts, among them J2 Screw_Terminal_01x02, J3 Screw_Terminal_01x02, Q1 NMOS, Q2 NMOS, U1 IR2184

Commit message: fixed kicad error
Parts:
- removed Vgs_Q1: Conn_01x02_Pin, Connector_PinHeader_2.54mm:PinHeader_1x02_P2.54mm_Vertical
- moved Q2 1.25 mm to (141.7, 92.0)
- moved Q1 1.20 mm to (126.2, 92.0)
Routing:
- net (no net): vias 0 -> 4

Commit message: fixed pcb
Parts:
- removed D2, D3: D_Schottky, Diode_THT:D_A-405_P7.62mm_Horizontal
- removed DQ1, DQ2, IL1: TestPoint, TestPoint:TestPoint_Bridge_Pitch2.54mm_Drill0.7mm
- added TP1: TestPoint, TestPoint:TestPoint_Bridge_Pitch5.08mm_Drill1.3mm, F.Cu at (128.8, 127.5)
Routing:
- net Net-(U1-HO): track 20.1 -> 0.00 mm
