File: Design/pcb/buck_bidireccional/buck_bidireccional.kicad_sch (KiCad schematic)
At the start: 24 parts, among them J2 Screw_Terminal_01x02, J3 Screw_Terminal_01x02, Q1 NMOS, Q2 NMOS, U1 IR2184

Commit message: fixed pcb
Parts:
- removed D2, D3: D_Schottky, Diode_THT:D_A-405_P7.62mm_Horizontal, symbol Device:D_Schottky
- removed DQ1, DQ2, IL1: TestPoint, TestPoint:TestPoint_Bridge_Pitch2.54mm_Drill0.7mm, symbol Connector:TestPoint
- added TP1: TestPoint, TestPoint:TestPoint_Bridge_Pitch5.08mm_Drill1.3mm, symbol Connector:TestPoint
Connections:
- net at C2.1, J2.1 (Pin_1), L1.1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: now also TP1.1
Other:
- moved on the sheet: R2, R3
