File: Design/pcb/final_pcb/untitled.kicad_sch (KiCad schematic)
At the start: 17 parts, among them J1 USB_C_Receptacle_USB2.0_14P, J5 Conn_01x05_Pin, U2 PIC32MZ2048EFM144-I/PH, U4 LM1117DT-3.3, Y1 SG-8002CA

Commit message: Final PCB
Parts:
- removed U4: LM1117DT-3.3, Package_TO_SOT_SMD:TO-252-3_TabPin2, symbol Regulator_Linear:LM1117DT-3.3
- added C14, C16, C17: 10u, Capacitor_SMD:C_1210_3225Metric, symbol Device:C
- added C15, C18: 0.1u, Capacitor_SMD:C_1210_3225Metric, symbol Device:C
- added L2: L, Inductor_SMD:L_1210_3225Metric, symbol Device:L
- added R10: 0, Resistor_SMD:R_0603_1608Metric_Pad0.98x0.95mm_HandSolder, symbol Device:R
- added R8: 6.19k, Resistor_SMD:R_1812_4532Metric, symbol Device:R
- added R9: 20k, Resistor_SMD:R_1812_4532Metric, symbol Device:R
- added U5: TPS560200, Package_TO_SOT_SMD:SOT-23-5, symbol Regulator_Switching:TPS560200
- J1: footprint Connector_USB:USB_C_Receptacle_GCT_USB4105-xx-A_16P_TopMnt_Horizontal -> Connector_USB:USB_C_Receptacle_GCT_USB4110
Connections:
- net 3.3V: now also C16.2, C17.2, C18.2, L2.2, R10.1, R10.2, R8.2
- net GND: now also C14.1, C15.1, C16.1, C17.1, R9.1, U5.2 (GND)
- new net: C18.1, R8.1, R9.2, U5.5 (FB)
- new net: L2.1, U5.3 (PH)
- new net 12v: C14.2, C15.2, U5.1 (EN), U5.4 (VIN)
- no-connect marks 0 -> 1
Other:
- moved on the sheet: J1, J5, R5, R6, R7
