File: Design/pcb/final_pcb/final_pcb.kicad_sch (KiCad schematic)
At the start: 16 parts, among them J2 Screw_Terminal_01x02, J3 Screw_Terminal_01x02, Q1 NMOS, Q2 NMOS, U1 IR2184, U3 LM7812_TO220

Commit message: Final PCB
Parts:
- J2, J3: footprint TerminalBlock_Phoenix:TerminalBlock_Phoenix_MKDS-1,5-2-5.08_1x02_P5.08mm_Horizontal -> TerminalBlock_Phoenix:TerminalBlock_Phoenix_PTSM-0,5-2-2,5-V-SMD_1x02-1MP_P2.50mm_Vertical
- U3: value LM7812_TO220 -> LM7812
Connections:
- net 5v renamed LM_input
Changed lines of the file:
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@@
 	)
 	(junction
-		(at 154.94 109.22)
+		(at 50.8 93.98)
 		(diameter 0)
 		(color 0 0 0 0)
@@
 	(wire
 		(pts
-			(xy 50.8 109.22) (xy 50.8 92.71)
+			(xy 50.8 109.22) (xy 50.8 93.98)
 		)
 		(stroke
@@
 	(wire
 		(pts
-			(xy 139.7 110.49) (xy 139.7 109.22)
+			(xy 43.18 93.98) (xy 50.8 93.98)
 		)
 		(stroke
@@
 	(wire
 		(pts
-			(xy 154.94 104.14) (xy 154.94 109.22)
-		)
-		(stroke
-			(width 0)
-			(type default)
-		)
-	)
-	(wire
-		(pts
 			(xy 200.66 99.06) (xy 200.66 105.41)
 		)
@@
 	(wire
 		(pts
-			(xy 139.7 109.22) (xy 154.94 109.22)
-		)
-		(stroke
-			(width 0)
-			(type default)
-		)
-	)
-	(wire
-		(pts
 			(xy 171.45 92.71) (xy 171.45 104.14)
 		)
@@
 	(wire
 		(pts
-			(xy 33.02 109.22) (xy 34.29 109.22)
+			(xy 24.13 109.22) (xy 34.29 109.22)
 		)
 		(stroke
@@
 	(wire
 		(pts
+			(xy 50.8 93.98) (xy 50.8 92.71)
+		)
+		(stroke
+			(width 0)
+			(type default)
+		)
+	)
+	(wire
+		(pts
 			(xy 64.77 130.81) (xy 77.47 130.81)
 		)
@@
 	(wire
 		(pts
-			(xy 154.94 109.22) (xy 154.94 120.65)
+			(xy 154.94 104.14) (xy 154.94 120.65)
 		)
 		(stroke
@@
 	(global_label "LM_input"
 		(shape input)
-		(at 33.02 109.22 180)
+		(at 24.13 109.22 180)
 		(fields_autoplaced yes)
 		(effects
@@
 		)
 		(property "Intersheetrefs" "${INTERSHEET_REFS}"
-			(at 21.8102 109.22 0)
+			(at 12.9202 109.22 0)
 			(effects
 				(font
@@
 		)
 	)
+	(global_label "12v"
+		(shape output)
+		(at 43.18 93.98 180)
+		(fields_autoplaced yes)
+		(effects
+			(font
+				(size 1.27 1.27)
+			)
+			(justify right)
+		)
+		(property "Intersheetrefs" "${INTERSHEET_REFS}"
+			(at 36.8082 93.98 0)
+			(effects
+				(font
+					(size 1.27 1.27)
+				)
+				(justify right)
+				(hide yes)
+			)
+		)
+	)
 	(global_label "VS"
 		(shape input)
@@
 				)
 				(justify left)
-				(hide yes)
-			)
-		)
-	)
-	(global_label "5v"
-		(shape output)
-		(at 139.7 110.49 180)
-		(fields_autoplaced yes)
-		(effects
-			(font
-				(size 1.27 1.27)
-			)
-			(justify right)
-		)
-		(property "Intersheetrefs" "${INTERSHEET_REFS}"
-			(at 134.5377 110.49 0)
-			(effects
-				(font
-					(size 1.27 1.27)
-				)
-				(justify right)
 				(hide yes)
 			)
@@
 			)
 		)
-		(property "Footprint" "TerminalBlock_Phoenix:TerminalBlock_Phoenix_MKDS-1,5-2-5.08_1x02_P5.08mm_Horizontal"
+		(property "Footprint" "TerminalBlock_Phoenix:TerminalBlock_Phoenix_PTSM-0,5-2-2,5-V-SMD_1x02-1MP_P2.50mm_Vertical"
 			(at 149.86 120.65 0)
 			(effects
@@
 			)
 		)
-		(property "Footprint" "TerminalBlock_Phoenix:TerminalBlock_Phoenix_MKDS-1,5-2-5.08_1x02_P5.08mm_Horizontal"
+		(property "Footprint" "TerminalBlock_Phoenix:TerminalBlock_Phoenix_PTSM-0,5-2-2,5-V-SMD_1x02-1MP_P2.50mm_Vertical"
 			(at 257.81 127 0)
 			(effects
@@
 			)
 		)
-		(property "Value" "LM7812_TO220"
+		(property "Value" "LM7812"
 			(at 41.91 105.41 0)
 			(effects

Commit message: pcb fix
Connections:
- net GND: no longer U1.2 (~{SD})
Changed lines of the file:
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@@
+	)
+	(junction
+		(at 49.53 149.86)
+		(diameter 0)
+		(color 0 0 0 0)
 	)
 	(junction
@@
 	)
 	(junction
-		(at 45.72 149.86)
-		(diameter 0)
-		(color 0 0 0 0)
-	)
-	(junction
 		(at 171.45 104.14)
 		(diameter 0)
@@
 		(color 0 0 0 0)
 	)
-	(junction
-		(at 45.72 138.43)
-		(diameter 0)
-		(color 0 0 0 0)
-	)
 	(wire
 		(pts
@@
 	(wire
 		(pts
-			(xy 45.72 149.86) (xy 57.15 149.86)
+			(xy 41.91 149.86) (xy 49.53 149.86)
 		)
 		(stroke
@@
 	(wire
 		(pts
+			(xy 49.53 149.86) (xy 57.15 149.86)
+		)
+		(stroke
+			(width 0)
+			(type default)
+		)
+	)
+	(wire
+		(pts
+			(xy 49.53 149.86) (xy 49.53 151.13)
+		)
+		(stroke
+			(width 0)
+			(type default)
+		)
+	)
+	(wire
+		(pts
 			(xy 64.77 128.27) (xy 69.85 128.27)
 		)
@@
 	(wire
 		(pts
-			(xy 45.72 138.43) (xy 49.53 138.43)
-		)
-		(stroke
-			(width 0)
-			(type default)
-		)
-	)
-	(wire
-		(pts
 			(xy 68.58 113.03) (xy 69.85 113.03)
 		)
@@
 	(wire
 		(pts
-			(xy 33.02 138.43) (xy 45.72 138.43)
-		)
-		(stroke
-			(width 0)
-			(type default)
-		)
-	)
-	(wire
-		(pts
 			(xy 24.13 109.22) (xy 34.29 109.22)
 		)
@@
 	(wire
 		(pts
-			(xy 45.72 138.43) (xy 45.72 149.86)
-		)
-		(stroke
-			(width 0)
-			(type default)
-		)
-	)
-	(wire
-		(pts
 			(xy 154.94 104.14) (xy 171.45 104.14)
 		)
@@
 		(pts
 			(xy 71.12 101.6) (xy 72.39 101.6)
-		)
-		(stroke
-			(width 0)
-			(type default)
-		)
-	)
-	(wire
-		(pts
-			(xy 41.91 149.86) (xy 45.72 149.86)
 		)
 		(stroke
@@
 	(global_label "GND"
 		(shape passive)
-		(at 33.02 138.43 180)
+		(at 49.53 151.13 270)
 		(fields_autoplaced yes)
 		(effects
@@
 		)
 		(property "Intersheetrefs" "${INTERSHEET_REFS}"
-			(at 27.2756 138.43 0)
+			(at 49.53 156.8744 90)
 			(effects
 				(font
